Commit message: Add warehouse SLAM and tugbot bridge updates

File: src/tugbot_description/urdf/tugbot_minimal.urdf.xacro (robot description, xacro)
@@ -15,69 +15,42 @@
   <link name="base_link">
     <visual>
-      <origin xyz="-0.10 0 0.10" rpy="0 0 0"/>
+      <origin xyz="0.155 0 0.3375" rpy="0 0 0"/>
       <geometry>
-        <box size="0.60 0.45 0.20"/>
+        <box size="1.204 0.754 0.239"/>
       </geometry>
       <material name="dark_gray"/>
     </visual>
     <collision>
-      <origin xyz="-0.10 0 0.10" rpy="0 0 0"/>
+      <origin xyz="0.155 0 0.3375" rpy="0 0 0"/>
       <geometry>
-        <box size="0.60 0.45 0.20"/>
+        <box size="1.204 0.754 0.239"/>
+      </geometry>
+    </collision>
+    <visual>
+      <origin xyz="-0.3266 0 0.532" rpy="0 0 0"/>
+      <geometry>
+        <box size="0.2408 0.754 0.15"/>
+      </geometry>
+      <material name="dark_gray"/>
+    </visual>
+    <collision>
+      <origin xyz="-0.3266 0 0.532" rpy="0 0 0"/>
+      <geometry>
+        <box size="0.2408 0.754 0.15"/>
       </geometry>
     </collision>
     <inertial>
-      <origin xyz="-0.10 0 0.10" rpy="0 0 0"/>
-      <mass value="46.2"/>
-      <inertia ixx="1.55925" ixy="0" ixz="0" iyy="1.55925" iyz="0" izz="1.55925"/>
+      <origin xyz="0.155 0 0.3375" rpy="0 0 0"/>
+      <mass value="43.0"/>
+      <inertia ixx="3.213" ixy="0" ixz="0" iyy="6.068" iyz="0" izz="7.541"/>
     </inertial>
-  </link>
-  <joint name="imu_link_joint" type="fixed">
-    <parent link="base_link"/>
-    <child link="imu_link"/>
-    <origin xyz="0.14 0.02 0.25" rpy="0 0 -1.57"/>
-  </joint>
-  <link name="imu_link">
-    <visual>
-      <geometry>
-        <box size="0.04 0.03 0.02"/>
-      </geometry>
-      <material name="sensor_black"/>
-    </visual>
-  </link>
-  <joint name="scan_front_joint" type="fixed">
-    <parent link="base_link"/>
-    <child link="scan_front"/>
-    <origin xyz="0.221 0 0.1404" rpy="0 0 0"/>
-  </joint>
-  <link name="scan_front">
-    <visual>
-      <geometry>
-        <cylinder radius="0.035" length="0.04"/>
-      </geometry>
-      <material name="sensor_black"/>
-    </visual>
-  </link>
-  <joint name="scan_back_joint" type="fixed">
-    <parent link="base_link"/>
-    <child link="scan_back"/>
-    <origin xyz="-0.2075 0 0.205" rpy="0 0 3.141592654"/>
-  </joint>
-  <link name="scan_back">
-    <visual>
-      <geometry>
-        <cylinder radius="0.035" length="0.04"/>
-      </geometry>
-      <material name="sensor_black"/>
-    </visual>
   </link>
   <joint name="scan_omni_joint" type="fixed">
     <parent link="base_link"/>
     <child link="scan_omni"/>
-    <origin xyz="-0.1855 0 0.5318" rpy="0 0 0"/>
+    <origin xyz="-0.3266 0 0.652" rpy="0 0 0"/>
   </joint>
   <link name="scan_omni">
     <visual>
-      <origin xyz="0 0 -0.035" rpy="0 0 0"/>
       <geometry>
         <cylinder radius="0.06" length="0.09"/>
